Commit message: Updated cog for ur16 how I understand the documentation
used documentation:
https://www.universal-robots.com/how-tos-and-faqs/faq/ur-faq/parameters-for-calculations-of-kinematics-and-dynamics-45257/

Note: This changes inertia for all robots as the main xacro file is changed.

File: ur_description/urdf/ur_macro.xacro (robot description, xacro)
@@ -107,5 +107,5 @@
       </collision>
       <xacro:cylinder_inertial radius="${shoulder_inertia_radius}" length="${shoulder_inertia_length}" mass="${shoulder_mass}">
-        <origin xyz="0 0 0" rpy="0 0 0" />
+        <origin xyz="${shoulder_cog}" rpy="0 0 0" />
       </xacro:cylinder_inertial>
     </link>
@@ -127,5 +127,5 @@
       </collision>
       <xacro:cylinder_inertial radius="${upperarm_inertia_radius}" length="${upperarm_inertia_length}" mass="${upper_arm_mass}">
-        <origin xyz="${-0.5 * upperarm_inertia_length} 0.0 ${upper_arm_inertia_offset}" rpy="0 ${pi/2} 0" />
+        <origin xyz="${upper_arm_cog}" rpy="0 ${pi/2} 0" />
       </xacro:cylinder_inertial>
     </link>
@@ -147,5 +147,5 @@
       </collision>
       <xacro:cylinder_inertial radius="${forearm_inertia_radius}" length="${forearm_inertia_length}"  mass="${forearm_mass}">
-        <origin xyz="${-0.5 * forearm_inertia_length} 0.0 ${elbow_offset}" rpy="0 ${pi/2} 0" />
+        <origin xyz="${forearm_cog}" rpy="0 ${pi/2} 0" />
       </xacro:cylinder_inertial>
     </link>
@@ -168,5 +168,5 @@
       </collision>
       <xacro:cylinder_inertial radius="${wrist_1_inertia_radius}" length="${wrist_1_inertia_length}"  mass="${wrist_1_mass}">
-        <origin xyz="0 0 0" rpy="0 0 0" />
+        <origin xyz="${wrist_1_cog}" rpy="0 0 0" />
       </xacro:cylinder_inertial>
     </link>
@@ -188,5 +188,5 @@
       </collision>
       <xacro:cylinder_inertial radius="${wrist_2_inertia_radius}" length="${wrist_2_inertia_length}"  mass="${wrist_2_mass}">
-        <origin xyz="0 0 0" rpy="0 0 0" />
+        <origin xyz="${wrist_2_cog}" rpy="0 0 0" />
       </xacro:cylinder_inertial>
     </link>
@@ -208,5 +208,5 @@
       </collision>
       <xacro:cylinder_inertial radius="${wrist_3_inertia_radius}" length="${wrist_3_inertia_length}"  mass="${wrist_3_mass}">
-        <origin xyz="0.0 0.0 ${-0.5 * wrist_3_inertia_length}" rpy="0 0 0" />
+        <origin xyz="${wrist_3_cog}" rpy="0 0 0" />
       </xacro:cylinder_inertial>
     </link>
