Commit message: Add extruder in urdf model

File: ur_description/urdf/ur3.urdf copy.xacro (robot description, xacro)
@@ -1,5 +1,5 @@
 <?xml version="1.0"?>
 <robot xmlns:xacro="http://wiki.ros.org/xacro">
-  <!--
+<!--
   Author: Felix Messmer
 -->
@@ -10,13 +10,23 @@
       <mass value="${mass}" />
       <xacro:insert_block name="origin" />
-      <inertia ixx="${0.0833333 * mass * (3 * radius * radius + length * length)}" ixy="0.0" ixz="0.0" iyy="${0.0833333 * mass * (3 * radius * radius + length * length)}" iyz="0.0" izz="${0.5 * mass * radius * radius}" />
+      <inertia ixx="${0.0833333 * mass * (3 * radius * radius + length * length)}" ixy="0.0" ixz="0.0"
+        iyy="${0.0833333 * mass * (3 * radius * radius + length * length)}" iyz="0.0"
+        izz="${0.5 * mass * radius * radius}" />
     </inertial>
   </xacro:macro>
-  <xacro:macro name="ur3_robot" params="prefix joint_limited shoulder_pan_lower_limit:=${-pi} shoulder_pan_upper_limit:=${pi} shoulder_lift_lower_limit:=${-pi} shoulder_lift_upper_limit:=${pi} elbow_joint_lower_limit:=${-pi} elbow_joint_upper_limit:=${pi} wrist_1_lower_limit:=${-pi} wrist_1_upper_limit:=${pi} wrist_2_lower_limit:=${-pi} wrist_2_upper_limit:=${pi} wrist_3_lower_limit:=${-pi} wrist_3_upper_limit:=${pi} transmission_hw_interface:=hardware_interface/PositionJointInterface safety_limits:=false safety_pos_margin:=0.15 safety_k_position:=20
+  <xacro:macro name="ur3_robot" params="prefix joint_limited
+    shoulder_pan_lower_limit:=${-pi}    shoulder_pan_upper_limit:=${pi}
+    shoulder_lift_lower_limit:=${-pi}    shoulder_lift_upper_limit:=${pi}
+    elbow_joint_lower_limit:=${-pi}    elbow_joint_upper_limit:=${pi}
+    wrist_1_lower_limit:=${-pi}    wrist_1_upper_limit:=${pi}
+    wrist_2_lower_limit:=${-pi}    wrist_2_upper_limit:=${pi}
+    wrist_3_lower_limit:=${-pi}    wrist_3_upper_limit:=${pi}
+    transmission_hw_interface:=hardware_interface/PositionJointInterface
+    safety_limits:=false safety_pos_margin:=0.15
+    safety_k_position:=20
     kinematics_file">
     <xacro:property name="__kinematics" value="${kinematics_file['kinematics']}"/>
     <!-- Inertia parameters -->
-    <xacro:property name="base_mass" value="2.0" />
-    <!-- This mass might be incorrect -->
+    <xacro:property name="base_mass" value="2.0" />  <!-- This mass might be incorrect -->
     <xacro:property name="shoulder_mass" value="2.0" />
     <xacro:property name="upper_arm_mass" value="3.42" />
@@ -36,13 +46,10 @@
     <xacro:property name="wrist_3_cog" value="0.0 0.0 -0.02" />
     <!-- Arbitrary offsets for shoulder/elbow joints -->
-    <xacro:property name="shoulder_offset" value="0.1198" />
-    <!-- measured from model -->
-    <xacro:property name="elbow_offset" value="0.0275" />
-    <!-- measured from model -->
-    <xacro:property name="upper_arm_inertia_offset" value="0.12" />
-    <!-- measured from model -->
+    <xacro:property name="shoulder_offset" value="0.1198" />  <!-- measured from model -->
+    <xacro:property name="elbow_offset" value="0.0275" /> <!-- measured from model -->
+    <xacro:property name="upper_arm_inertia_offset" value="0.12" />  <!-- measured from model -->
     <!-- This is for compatibility reasons, as transformation between base and base_link was always 180 degree in the ur_description -->
     <xacro:property name="base_correction" value="${pi}" />
-    <link name="${prefix}base_link">
+    <link name="${prefix}base_link" >
       <visual>
         <origin xyz="0 0 0" rpy="0 0 ${base_correction}"/>
@@ -301,28 +308,16 @@
       <parent link="${prefix}wrist_3_link" />
       <child link = "${prefix}ee_link" />
-      <origin xyz="-0.036 0.069 -0.054" rpy="0.0 0.0 0.0" />
+      <origin xyz="0.0 0.0 0.0" rpy="0.0 ${-pi/2.0} ${pi/2.0}" />
     </joint>
     <link name="${prefix}ee_link">
-      <visual>
-        <origin xyz="0 0 0" rpy="${pi/2} 0 0"/>
-        <geometry>
-          <mesh filename="package://ur_description/meshes/ur3/collision/extruder.stl"/>
-        </geometry>
-        <material name="LightGrey">
-          <color rgba="0.7 0.7 0.7 1.0"/>
-        </material>
-      </visual>
-      <collision>
-        <origin xyz="0 0 0" rpy="${pi/2} 0 0"/>
-        <geometry>
-          <mesh filename="package://ur_description/meshes/ur3/collision/extruder.stl"/>
-        </geometry>
-      </collision>
-      <xacro:cylinder_inertial radius="0.045" length="0.0305" mass="${wrist_3_mass}">
-        <origin xyz="0.0 0.0 ${-0.0305/2}" rpy="0 0 0" />
-      </xacro:cylinder_inertial>
+      <collision>
+        <geometry>
+          <box size="0.01 0.01 0.01"/>
+        </geometry>
+        <origin rpy="0 0 0" xyz="-0.01 0 0"/>
+      </collision>
     </link>
     <joint name="${prefix}wrist_3_passive_joint" type="fixed">
-      <origin xyz="0 0 0.108" rpy="0.0 ${-pi/2.0} ${pi/2.0}"/>
+      <origin xyz="0 0 0" rpy="0 0 0"/>
       <parent link="${prefix}wrist_3_link"/>
       <child link="${prefix}tool0"/>
