Commit message: Add extruder in robot urdf model

File: ur_description/urdf/ur3.urdf.xacro (robot description, xacro)
@@ -336,6 +336,4 @@
       <child link="${prefix}base"/>
     </joint>
-    <!-- Frame coincident with all-zeros TCP on UR controller -->
-    <link name="${prefix}tool0"/>
   </xacro:macro>
 </robot>

Commit message: Add extruder to the wirst3 link

File: ur_description/urdf/ur3.urdf.xacro (robot description, xacro)
@@ -301,5 +301,5 @@
       <parent link="${prefix}wrist_3_link" />
       <child link = "${prefix}ee_link" />
-      <origin xyz="-0.036 0.069 -0.054" rpy="0.0 0.0 0.0" />
+      <origin xyz="-0.036 0.069 -0.0545" rpy="0.0 0.0 0.0" />
     </joint>
     <link name="${prefix}ee_link">
@@ -323,6 +323,7 @@
       </xacro:cylinder_inertial>
     </link>
+    <!-- Defines the TCP position -->
     <joint name="${prefix}wrist_3_passive_joint" type="fixed">
-      <origin xyz="0 0 0.108" rpy="0.0 ${-pi/2.0} ${pi/2.0}"/>
+      <origin xyz="-0.001 0.046 0.109" rpy="0.0 ${-pi/2.0} ${pi/2.0}"/>
       <parent link="${prefix}wrist_3_link"/>
       <child link="${prefix}tool0"/>

Commit message: some params edit work

File: ur_description/urdf/ur3.urdf.xacro (robot description, xacro)
@@ -325,5 +325,5 @@
     <!-- Defines the TCP position -->
     <joint name="${prefix}wrist_3_passive_joint" type="fixed">
-      <origin xyz="-0.001 0.046 0.109" rpy="0.0 ${-pi/2.0} ${pi/2.0}"/>
+      <origin xyz="0.00047 0.00076 0.11311" rpy="0.0 ${-pi/2.0} ${pi/2.0}"/>
       <parent link="${prefix}wrist_3_link"/>
       <child link="${prefix}tool0"/>

Commit message: Update work

File: ur_description/urdf/ur3.urdf.xacro (robot description, xacro)
@@ -325,5 +325,5 @@
     <!-- Defines the TCP position -->
     <joint name="${prefix}wrist_3_passive_joint" type="fixed">
-      <origin xyz="0.00047 0.00076 0.11311" rpy="0.0 ${-pi/2.0} ${pi/2.0}"/>
+      <origin xyz="0.03605 0.01281 0.11147" rpy="0.0 ${-pi/2.0} ${pi/2.0}"/>
       <parent link="${prefix}wrist_3_link"/>
       <child link="${prefix}tool0"/>
